Commit message: camera_package

File: robotic_arm_description/urdf/robotic_arm_urdf.urdf (robot description, URDF)
Before this commit: robot robotic_arm, 13 links, 12 joints
Links:
- removed link gripper_finger_1
- removed link gripper_finger_2
- added link end_effector
- link gripper_base: geometry collision box size=0.08 0.01 0.01; visual box size=0.08 0.01 0.01
Joints:
- removed joint left_gripper_joint
- removed joint right_gripper_joint
- added joint end_effector_link: type fixed, parent gripper_base, child end_effector, origin xyz= 0 -0.08 0  rpy=0 0 0
