Commit message: Update on the robot work station

File: robotic_arm_description/urdf/materials.xacro (robot description, xacro)
@@ -4,9 +4,12 @@
   <color rgba="0.700 0.700 0.700 1.000"/>
 </material>
-<material name="oak">
-  <color rgba="0.7098 0.5882 0.4431 1.000"/>
+<material name="led_red">
+  <color rgba="0.7686274509803922 0.20784313725490197 0.15294117647058825 1.0"/>
 </material>
 <material name="pa_12_nylon_pa_603cf_with_eos_p_3d_printers">
   <color rgba="0.24705882352941178 0.24705882352941178 0.24705882352941178 1.0"/>
 </material>
+<material name = "oak">
+  <color rgba = "0.8157 0.6510 0.4902 1.0 "/>
+</material>
 </robot>

File: robotic_arm_description/urdf/robotic_arm.xacro (robot description, xacro)
@@ -2,5 +2,4 @@
 <robot name="robotic_arm" xmlns:xacro="http://www.ros.org/wiki/xacro">
 <!-- Load Simulated or Real Hardware Interfaces -->
-<xacro:arg name="is_sim" default="true"/>
 <xacro:include filename="$(find robotic_arm_description)/urdf/materials.xacro" />
 <xacro:include filename="$(find robotic_arm_description)/urdf/robotic_arm.trans" />
@@ -8,12 +7,12 @@
 <xacro:include filename="$(find robotic_arm_description)/urdf/robotic_arm_controllers.xacro"/>
 <!-- Properties -->
-<xacro:property name="PI" value="1.570796"/>\
+<xacro:property name="PI" value="1.570796"/>
 <!-- Links -->
 <link name = "world"/>
 <link name="base_link">
   <inertial>
-    <origin xyz="4.1292719567255465e-17 -0.1275 0.0075" rpy="0 0 0"/>
-    <mass value="2.5408670074548567"/>
-    <inertia ixx="0.033061" iyy="0.074955" izz="0.107921" ixy="-0.0" iyz="0.0" ixz="0.0"/>
+    <origin xyz="2.5964963671146073e-05 -0.12750519341019426 0.02735001860163422" rpy="0 0 0"/>
+    <mass value="2.562361438794821"/>
+    <inertia ixx="0.033829" iyy="0.076749" izz="0.110468" ixy="-2e-06" iyz="0.0" ixz="-0.0"/>
   </inertial>
   <visual>
@@ -31,12 +30,92 @@
   </collision>
 </link>
+<link name="container_1">
+  <inertial>
+    <origin xyz="0.0021344768560282723 -1.5647124724599282e-05 0.026103286200414536" rpy="0 0 0"/>
+    <mass value="0.8859344258495231"/>
+    <inertia ixx="0.002047" iyy="0.003759" izz="0.004728" ixy="1e-06" iyz="0.0" ixz="0.000223"/>
+  </inertial>
+  <visual>
+    <origin xyz="0.2025 0.225 -0.035" rpy="0 0 0"/>
+    <geometry>
+      <mesh filename="package://robotic_arm_description/meshes/container_1.stl" scale="0.001 0.001 0.001"/>
+    </geometry>
+    <material name="led_red"/>
+  </visual>
+  <collision>
+    <origin xyz="0.2025 0.225 -0.035" rpy="0 0 0"/>
+    <geometry>
+      <mesh filename="package://robotic_arm_description/meshes/container_1.stl" scale="0.001 0.001 0.001"/>
+    </geometry>
+  </collision>
+</link>
+<link name="container_2">
+  <inertial>
+    <origin xyz="-1.565155782010108e-05 -0.0021344802460424653 0.026103286200414424" rpy="0 0 0"/>
+    <mass value="0.8859344258495231"/>
+    <inertia ixx="0.003759" iyy="0.002047" izz="0.004728" ixy="-1e-06" iyz="-0.000223" ixz="0.0"/>
+  </inertial>
+  <visual>
+    <origin xyz="0.2425 0.02 -0.035" rpy="0 0 0"/>
+    <geometry>
+      <mesh filename="package://robotic_arm_description/meshes/container_2.stl" scale="0.001 0.001 0.001"/>
+    </geometry>
+    <material name="led_red"/>
+  </visual>
+  <collision>
+    <origin xyz="0.2425 0.02 -0.035" rpy="0 0 0"/>
+    <geometry>
+      <mesh filename="package://robotic_arm_description/meshes/container_2.stl" scale="0.001 0.001 0.001"/>
+    </geometry>
+  </collision>
+</link>
+<link name="container_3">
+  <inertial>
+    <origin xyz="-1.565155782010108e-05 -0.0021344802460424445 0.0261032862004145" rpy="0 0 0"/>
+    <mass value="0.8859344258495231"/>
+    <inertia ixx="0.003759" iyy="0.002047" izz="0.004728" ixy="-1e-06" iyz="-0.000223" ixz="0.0"/>
+  </inertial>
+  <visual>
+    <origin xyz="0.1375 0.02 -0.035" rpy="0 0 0"/>
+    <geometry>
+      <mesh filename="package://robotic_arm_description/meshes/container_3.stl" scale="0.001 0.001 0.001"/>
+    </geometry>
+    <material name="led_red"/>
+  </visual>
+  <collision>
+    <origin xyz="0.1375 0.02 -0.035" rpy="0 0 0"/>
+    <geometry>
+      <mesh filename="package://robotic_arm_description/meshes/container_3.stl" scale="0.001 0.001 0.001"/>
+    </geometry>
+  </collision>
+</link>
+<link name="camera_support">
+  <inertial>
+    <origin xyz="8.696769445861888e-16 -0.01380572988450951 0.19182498575975282" rpy="0 0 0"/>
+    <mass value="1.9073849170892592"/>
+    <inertia ixx="0.059599" iyy="0.059727" izz="0.000405" ixy="-0.0" iyz="0.000448" ixz="0.0"/>
+  </inertial>
+  <visual>
+    <origin xyz="-0.0 0.325 -0.02" rpy="0 0 0"/>
+    <geometry>
+      <mesh filename="package://robotic_arm_description/meshes/camera_support.stl" scale="0.001 0.001 0.001"/>
+    </geometry>
+    <material name="pa_12_nylon_pa_603cf_with_eos_p_3d_printers"/>
+  </visual>
+  <collision>
+    <origin xyz="-0.0 0.325 -0.02" rpy="0 0 0"/>
+    <geometry>
+      <mesh filename="package://robotic_arm_description/meshes/camera_support.stl" scale="0.001 0.001 0.001"/>
+    </geometry>
+  </collision>
+</link>
 <link name="base">
   <inertial>
-    <origin xyz="3.3070895591155684e-07 -0.06999939486232219 0.051365620594267386" rpy="0 0 0"/>
+    <origin xyz="6.051376774735407e-07 -0.08000032966587473 0.05136562059426733" rpy="0 0 0"/>
     <mass value="0.5102582987586253"/>
-    <inertia ixx="0.001541" iyy="0.00162" izz="0.002267" ixy="0.0" iyz="0.0" ixz="0.0"/>
-  </inertial>
-  <visual>
-    <origin xyz="-0.0 -0.07 -0.015" rpy="0 0 0"/>
+    <inertia ixx="0.00162" iyy="0.001541" izz="0.002267" ixy="-0.0" iyz="-0.0" ixz="0.0"/>
+  </inertial>
+  <visual>
+    <origin xyz="-0.0 -0.07 -0.035" rpy="0 0 0"/>
     <geometry>
       <mesh filename="package://robotic_arm_description/meshes/base.stl" scale="0.001 0.001 0.001"/>
@@ -45,5 +124,5 @@
   </visual>
   <collision>
-    <origin xyz="-0.0 -0.07 -0.015" rpy="0 0 0"/>
+    <origin xyz="-0.0 -0.07 -0.035" rpy="0 0 0"/>
     <geometry>
       <mesh filename="package://robotic_arm_description/meshes/base.stl" scale="0.001 0.001 0.001"/>
@@ -53,10 +132,10 @@
 <link name="waist">
   <inertial>
-    <origin xyz="-0.013899791072812253 -0.003284120079222943 0.02372142968591144" rpy="0 0 0"/>
+    <origin xyz="-0.013899791072812993 -0.0032841190361416073 0.023721429685911427" rpy="0 0 0"/>
     <mass value="0.11734363935702768"/>
     <inertia ixx="8.6e-05" iyy="7.9e-05" izz="8.5e-05" ixy="-3e-06" iyz="1.1e-05" ixz="1.4e-05"/>
   </inertial>
   <visual>
-    <origin xyz="0.0 0.0 -0.101" rpy="0 0 0"/>
+    <origin xyz="0.0 0.01 -0.121" rpy="0 0 0"/>
     <geometry>
       <mesh filename="package://robotic_arm_description/meshes/waist.stl" scale="0.001 0.001 0.001"/>
@@ -65,5 +144,5 @@
   </visual>
   <collision>
-    <origin xyz="0.0 0.0 -0.101" rpy="0 0 0"/>
+    <origin xyz="0.0 0.01 -0.121" rpy="0 0 0"/>
     <geometry>
       <mesh filename="package://robotic_arm_description/meshes/waist.stl" scale="0.001 0.001 0.001"/>
@@ -73,10 +152,10 @@
 <link name="link_1">
   <inertial>
-    <origin xyz="0.007817729878361625 -4.0523557253042963e-07 0.06000021649587692" rpy="0 0 0"/>
+    <origin xyz="0.007817729878360883 -4.041924911227235e-07 0.06000021649587681" rpy="0 0 0"/>
     <mass value="0.07112302510728019"/>
     <inertia ixx="0.000121" iyy="0.000116" izz="1e-05" ixy="0.0" iyz="-0.0" ixz="0.0"/>
   </inertial>
   <visual>
-    <origin xyz="0.001 0.014069 -0.141262" rpy="0 0 0"/>
+    <origin xyz="0.001 0.024069 -0.161262" rpy="0 0 0"/>
     <geometry>
       <mesh filename="package://robotic_arm_description/meshes/link_1.stl" scale="0.001 0.001 0.001"/>
@@ -85,5 +164,5 @@
   </visual>
   <collision>
-    <origin xyz="0.001 0.014069 -0.141262" rpy="0 0 0"/>
+    <origin xyz="0.001 0.024069 -0.161262" rpy="0 0 0"/>
     <geometry>
       <mesh filename="package://robotic_arm_description/meshes/link_1.stl" scale="0.001 0.001 0.001"/>
@@ -93,10 +172,10 @@
 <link name="link_2">
   <inertial>
-    <origin xyz="-0.01594540180295605 -0.046193837589282 4.672518474457821e-05" rpy="0 0 0"/>
+    <origin xyz="-0.015945401802956827 -0.04619383654620061 4.672518474435616e-05" rpy="0 0 0"/>
     <mass value="0.11456681455688399"/>
     <inertia ixx="0.000224" iyy="2.7e-05" izz="0.00023" ixy="2.7e-05" iyz="0.0" ixz="-0.0"/>
   </inertial>
   <visual>
-    <origin xyz="0.001 0.014069 -0.261262" rpy="0 0 0"/>
+    <origin xyz="0.001 0.024069 -0.281262" rpy="0 0 0"/>
     <geometry>
       <mesh filename="package://robotic_arm_description/meshes/link_2.stl" scale="0.001 0.001 0.001"/>
@@ -105,5 +184,5 @@
   </visual>
   <collision>
-    <origin xyz="0.001 0.014069 -0.261262" rpy="0 0 0"/>
+    <origin xyz="0.001 0.024069 -0.281262" rpy="0 0 0"/>
     <geometry>
       <mesh filename="package://robotic_arm_description/meshes/link_2.stl" scale="0.001 0.001 0.001"/>
@@ -113,10 +192,10 @@
 <link name="gripper_base">
   <inertial>
-    <origin xyz="0.016989765812988437 -0.03097536759348493 0.0043010847265131935" rpy="0 0 0"/>
+    <origin xyz="0.016989765812987632 -0.030975366550403616 0.004301084726513138" rpy="0 0 0"/>
     <mass value="0.02850874527831614"/>
     <inertia ixx="1e-05" iyy="7e-06" izz="1.4e-05" ixy="3e-06" iyz="1e-06" ixz="1e-06"/>
   </inertial>
   <visual>
-    <origin xyz="-0.00285 0.131419 -0.261562" rpy="0 0 0"/>
+    <origin xyz="-0.00285 0.141419 -0.281562" rpy="0 0 0"/>
     <geometry>
       <mesh filename="package://robotic_arm_description/meshes/gripper_base.stl" scale="0.001 0.001 0.001"/>
@@ -125,5 +204,5 @@
   </visual>
   <collision>
-    <origin xyz="-0.00285 0.131419 -0.261562" rpy="0 0 0"/>
+    <origin xyz="-0.00285 0.141419 -0.281562" rpy="0 0 0"/>
     <geometry>
       <mesh filename="package://robotic_arm_description/meshes/gripper_base.stl" scale="0.001 0.001 0.001"/>
@@ -133,10 +212,10 @@
 <link name="gripper_finger_1">
   <inertial>
-    <origin xyz="0.0025925452739243675 -0.04003700818287059 0.002000392615642277" rpy="0 0 0"/>
+    <origin xyz="0.0025925452739234515 -0.04003700713978928 0.0020003926156425544" rpy="0 0 0"/>
     <mass value="0.00844478254120791"/>
-    <inertia ixx="7e-06" iyy="0.0" izz="8e-06" ixy="1e-06" iyz="0.0" ixz="0.0"/>
-  </inertial>
-  <visual>
-    <origin xyz="-0.02875 0.169419 -0.276912" rpy="0 0 0"/>
+    <inertia ixx="7e-06" iyy="0.0" izz="8e-06" ixy="1e-06" iyz="-0.0" ixz="0.0"/>
+  </inertial>
+  <visual>
+    <origin xyz="-0.02875 0.179419 -0.295562" rpy="0 0 0"/>
     <geometry>
       <mesh filename="package://robotic_arm_description/meshes/gripper_finger_1.stl" scale="0.001 0.001 0.001"/>
@@ -145,5 +224,5 @@
   </visual>
   <collision>
-    <origin xyz="-0.02875 0.169419 -0.276912" rpy="0 0 0"/>
+    <origin xyz="-0.02875 0.179419 -0.295562" rpy="0 0 0"/>
     <geometry>
       <mesh filename="package://robotic_arm_description/meshes/gripper_finger_1.stl" scale="0.001 0.001 0.001"/>
@@ -153,10 +232,10 @@
 <link name="gripper_finger_2">
   <inertial>
-    <origin xyz="-0.00259254527392403 -0.04003700818287059 0.002000392615642388" rpy="0 0 0"/>
+    <origin xyz="-0.002592545273924804 -0.04003700713978928 0.002000392615642499" rpy="0 0 0"/>
     <mass value="0.00844478254120791"/>
-    <inertia ixx="7e-06" iyy="0.0" izz="8e-06" ixy="-1e-06" iyz="0.0" ixz="-0.0"/>
-  </inertial>
-  <visual>
-    <origin xyz="-0.00185 0.169419 -0.275562" rpy="0 0 0"/>
+    <inertia ixx="7e-06" iyy="0.0" izz="8e-06" ixy="-1e-06" iyz="-0.0" ixz="-0.0"/>
+  </inertial>
+  <visual>
+    <origin xyz="-0.00185 0.179419 -0.295562" rpy="0 0 0"/>
     <geometry>
       <mesh filename="package://robotic_arm_description/meshes/gripper_finger_2.stl" scale="0.001 0.001 0.001"/>
@@ -165,5 +244,5 @@
   </visual>
   <collision>
-    <origin xyz="-0.00185 0.169419 -0.275562" rpy="0 0 0"/>
+    <origin xyz="-0.00185 0.179419 -0.295562" rpy="0 0 0"/>
     <geometry>
       <mesh filename="package://robotic_arm_description/meshes/gripper_finger_2.stl" scale="0.001 0.001 0.001"/>
@@ -177,14 +256,33 @@
 </joint>
 <joint name="rigid_1" type="fixed">
-  <origin xyz="0.0 0.07 0.015" rpy="0 0 0"/>
+  <origin xyz="0.0 0.07 0.035" rpy="0 0 0"/>
   <parent link="base_link"/>
   <child link="base"/>
 </joint>
+<joint name="rigid_2" type="fixed">
+  <origin xyz="-0.2025 -0.225 0.035" rpy="0 0 0"/>
+  <parent link="base_link"/>
+  <child link="container_1"/>
+</joint>
+<joint name="rigid_3" type="fixed">
+  <origin xyz="-0.2425 -0.02 0.035" rpy="0 0 0"/>
+  <parent link="base_link"/>
+  <child link="container_2"/>
+</joint>
+<joint name="rigid_4" type="fixed">
+  <origin xyz="-0.1375 -0.02 0.035" rpy="0 0 0"/>
+  <parent link="base_link"/>
+  <child link="container_3"/>
+</joint>
+<joint name="rigid_5" type="fixed">
+  <origin xyz="0.0 -0.325 0.02" rpy="0 0 0"/>
+  <parent link="base_link"/>
+  <child link="camera_support"/>
+</joint>
 <joint name="base_waist_joint" type="revolute">
-  <origin xyz="-0.0 -0.07 0.086" rpy="0 0 0"/>
+  <origin xyz="-0.0 -0.08 0.086" rpy="0 0 0"/>
   <parent link="base"/>
   <child link="waist"/>
-  <axis xyz="0.0 0.0 1.0"/>
-  <dynamics damping="10.0" friction="2.0"/>
+  <axis xyz="-0.0 -0.0 1.0"/>
   <limit upper="1.570796" lower="-1.570796" effort="100" velocity="100"/>
 </joint>
@@ -194,5 +292,4 @@
   <child link="link_1"/>
   <axis xyz="1.0 0.0 -0.0"/>
-  <dynamics damping="10.0" friction="2.0"/>
   <limit upper="1.570796" lower="-1.570796" effort="100" velocity="100"/>
 </joint>
@@ -201,32 +298,29 @@
   <parent link="link_1"/>
   <child link="link_2"/>
-  <axis xyz="-1.0 0.0 -0.0"/>
-  <dynamics damping="10.0" friction="2.0"/>
-  <limit upper="3.141593" lower="0.0" effort="100" velocity="100"/>
-</joint>
-<joint name="link2_gripper_base_joint" type="revolute">
+  <axis xyz="1.0 -0.0 -0.0"/>
+  <limit upper="1.570796" lower="-1.570796" effort="100" velocity="100"/>
+</joint>
+<joint name="link2_gipper_base_joint" type="revolute">
   <origin xyz="0.00385 -0.11735 0.0003" rpy="0 0 0"/>
   <parent link="link_2"/>
   <child link="gripper_base"/>
-  <axis xyz="1.0 0.0 0.0"/>
-  <dynamics damping="10.0" friction="2.0"/>
+  <axis xyz="1.0 -0.0 0.0"/>
   <limit upper="1.570796" lower="-1.570796" effort="100" velocity="100"/>
 </joint>
 <joint name="right_gripper_joint" type="revolute">
+  <origin xyz="0.0259 -0.038 0.014" rpy="0 0 0"/>
+  <parent link="gripper_base"/>
+  <child link="gripper_finger_1"/>
+  <axis xyz="-0.0 0.0 1.0"/>
+  <limit upper="1.047198" lower="0.0" effort="100" velocity="100"/>
+</joint>
+<joint name="left_gripper_joint" type="revolute">
   <origin xyz="-0.001 -0.038 0.014" rpy="0 0 0"/>
   <parent link="gripper_base"/>
   <child link="gripper_finger_2"/>
-  <axis xyz="0.0 0.0 -1.0"/>
+  <axis xyz="-0.0 0.0 1.0"/>
   <dynamics damping="10.0" friction="2.0"/>
-  <limit upper="0.785398" lower="0.0" effort="100" velocity="100"/>
-</joint>
-<joint name="left_gripper_joint" type="revolute">
-  <origin xyz="0.0259 -0.038 0.01535" rpy="0 0 0"/>
-  <parent link="gripper_base"/>
-  <child link="gripper_finger_1"/>
-  <axis xyz="-0.0 -0.0 1.0"/>
-  <dynamics damping="10.0" friction="2.0"/>
-  <mimic joint = "right_gripper_joint" multiplier = "1.0"/>
-  <limit upper="-0.785398" lower="0.0" effort="100" velocity="100"/>
+  <mimic joint = "right_gripper_joint" multiplier = "-1.0"/>
+  <limit upper="0.0" lower="-1.047198" effort="100" velocity="100"/>
 </joint>
 </robot>

File: robotic_arm_description/urdf/robotic_arm_controllers.xacro (robot description, xacro)
@@ -3,17 +3,16 @@
 <xacro:property name="gripper_angle" value="0.7854"/>
 <xacro:property name="PI" value="3.14159"/>
-<xacro:if value = "$(arg is_sim)">
-    <hardware>
+ <!-- Gazebo Plugin -->
+ <gazebo>
+        <plugin filename="libgazebo_ros2_control.so" name="gazebo_ros2_control">
+            <robot_param> robot_description</robot_param>
+            <robot_param_node> robot_state_publisher</robot_param_node>
+            <parameters>$(find robotic_arm_controllers)/config/robot_arm_controllers.yaml</parameters>
+        </plugin>
+</gazebo>
+<ros2_control type = "system" name = "RoboticArmSystem">
+     <hardware>
         <plugin>gazebo_ros2_control/GazeboSystem</plugin>
     </hardware>
-</xacro:if>
-<xacro:unless value = "$(arg is_sim)">
-    <hardware>
-        <plugin>robotic_arm_hw/RoboticArmHWInterface</plugin>
-        <!-- Change the port here -->
-        <param name ="port">/dev/ttyUSB0</param>
-    </hardware>
-</xacro:unless>
-<ros2_control type = "system" name = "RoboticArmSystem">
 <!-- Interfaces -->
     <joint name="base_waist_joint">

File: robotic_arm_description/urdf/robotic_arm_gazebo.xacro (robot description, xacro)
@@ -6,62 +6,80 @@
 <xacro:property name="link_2_color" value = "Gazebo/FlatBlack" />
 <xacro:property name="gripper_base_color" value = "Gazebo/FlatBlack" />
-<xacro:property name="motor_color" value="Gazebo/Blue" />
 <xacro:property name="gripper_gears" value="GazeboGrey"/>
-<xacro:property name="gripper_color" value="Gazebo/DarkGrey" />
-<gazebo>
-        <plugin filename="libgazebo_ros2_control.so" name="gazebo_ros2_control">
-            <robot_param> robot_description</robot_param>
-            <robot_param_node> robot_state_publisher</robot_param_node>
-            <parameters>$(find robotic_arm_controllers)/config/robot_arm_controllers.yaml</parameters>
-        </plugin>
-</gazebo>
-<gazebo reference="base_link">
-  <material>${base_color}</material>
-  <mu1>0.2</mu1>
-  <mu2>0.2</mu2>
-  <self_collide>true</self_collide>
-  <gravity>true</gravity>
-</gazebo>
-<gazebo reference="base">
-  <material>${waist_color}</material>
-  <mu1>0.2</mu1>
-  <mu2>0.2</mu2>
-  <self_collide>true</self_collide>
-</gazebo>
-<gazebo reference="waist">
-  <material>${waist_color}</material>
-  <mu1>0.2</mu1>
-  <mu2>0.2</mu2>
-  <self_collide>true</self_collide>
-</gazebo>
-<gazebo reference="link_1">
-  <material>${link_1_color}</material>
-  <mu1>0.2</mu1>
-  <mu2>0.2</mu2>
-  <self_collide>true</self_collide>
-</gazebo>
-<gazebo reference="link_2">
-  <material>${link_2_color}</material>
-  <mu1>0.2</mu1>
-  <mu2>0.2</mu2>
-  <self_collide>true</self_collide>
-</gazebo>
-<gazebo reference="gripper_base">
-  <material>${gripper_base_color}</material>
-  <mu1>0.2</mu1>
-  <mu2>0.2</mu2>
-  <self_collide>true</self_collide>
-</gazebo>
-<gazebo reference="gripper_finger_1">
-  <material>${gripper_gears}</material>
-  <mu1>0.2</mu1>
-  <mu2>0.2</mu2>
-  <self_collide>true</self_collide>
-</gazebo>
-<gazebo reference="gripper_finger_2">
-  <material>${gripper_gears}</material>
-  <mu1>0.2</mu1>
-  <mu2>0.2</mu2>
-  <self_collide>true</self_collide>
-</gazebo>
+<xacro:property name="gripper_color" value="Gazebo/DarkGrey"/>
+<xacro:property name="camera_color" value="Gazebo/Oak" />
+<xacro:property name="container_color" value="Gazebo/Red" />
+  <gazebo reference="base_link">
+    <material>${base_color}</material>
+    <mu1>0.2</mu1>
+    <mu2>0.2</mu2>
+    <self_collide>true</self_collide>
+    <gravity>true</gravity>
+  </gazebo>
+  <gazebo reference="base">
+    <material>${waist_color}</material>
+    <mu1>0.2</mu1>
+    <mu2>0.2</mu2>
+    <self_collide>true</self_collide>
+  </gazebo>
+  <gazebo reference="waist">
+    <material>${waist_color}</material>
+    <mu1>0.2</mu1>
+    <mu2>0.2</mu2>
+    <self_collide>true</self_collide>
+  </gazebo>
+  <gazebo reference="link_1">
+    <material>${link_1_color}</material>
+    <mu1>0.2</mu1>
+    <mu2>0.2</mu2>
+    <self_collide>true</self_collide>
+  </gazebo>
+  <gazebo reference="link_2">
+    <material>${link_2_color}</material>
+    <mu1>0.2</mu1>
+    <mu2>0.2</mu2>
+    <self_collide>true</self_collide>
+  </gazebo>
+  <gazebo reference="gripper_base">
+    <material>${gripper_base_color}</material>
+    <mu1>0.2</mu1>
+    <mu2>0.2</mu2>
+    <self_collide>true</self_collide>
+  </gazebo>
+  <gazebo reference="gripper_finger_1">
+    <material>${gripper_gears}</material>
+    <mu1>0.2</mu1>
+    <mu2>0.2</mu2>
+    <self_collide>true</self_collide>
+  </gazebo>
+  <gazebo reference="gripper_finger_2">
+    <material>${gripper_gears}</material>
+    <mu1>0.2</mu1>
+    <mu2>0.2</mu2>
+    <self_collide>true</self_collide>
+  </gazebo>
+  <gazebo reference="camera_support">
+    <material>${camera_color}</material>
+    <mu1>0.2</mu1>
+    <mu2>0.2</mu2>
+    <self_collide>true</self_collide>
+  </gazebo>
+  <gazebo reference="container_1">
+    <material>${container_color}</material>
+    <mu1>0.2</mu1>
+    <mu2>0.2</mu2>
+    <self_collide>true</self_collide>
+  </gazebo>
+  <gazebo reference="container_2">
+    <material>${container_color}</material>
+    <mu1>0.2</mu1>
+    <mu2>0.2</mu2>
+    <self_collide>true</self_collide>
+  </gazebo>
+  <gazebo reference="container_3">
+    <material>${container_color}</material>
+    <mu1>0.2</mu1>
+    <mu2>0.2</mu2>
+    <self_collide>true</self_collide>
+  </gazebo>
 </robot>
