Commit message: __

File: robotic_arm_description/urdf/materials.xacro (robot description, xacro)
@@ -7,5 +7,5 @@
   <color rgba="0.7686274509803922 0.20784313725490197 0.15294117647058825 1.0"/>
 </material>
-<material name="pa_12_nylon_pa_603cf_with_eos_p_3d_printers">
+<material name="black_3d_printed">
   <color rgba="0.24705882352941178 0.24705882352941178 0.24705882352941178 1.0"/>
 </material>
@@ -13,3 +13,6 @@
   <color rgba = "0.8157 0.6510 0.4902 1.0 "/>
 </material>
+<material name="steel_satin">
+  <color rgba="0.6274509803921569 0.6274509803921569 0.6274509803921569 1.0"/>
+</material>
 </robot>

File: robotic_arm_description/urdf/robotic_arm.xacro (robot description, xacro)
@@ -96,21 +96,43 @@
 <link name="camera_support">
   <inertial>
-    <origin xyz="8.696769445861888e-16 -0.01380572988450951 0.19182498575975282" rpy="0 0 0"/>
-    <mass value="1.9073849170892592"/>
-    <inertia ixx="0.059599" iyy="0.059727" izz="0.000405" ixy="-0.0" iyz="0.000448" ixz="0.0"/>
-  </inertial>
-  <visual>
-    <origin xyz="-0.0 0.325 -0.02" rpy="0 0 0"/>
+    <origin xyz="-0.018363826080468604 -0.008283937089531401 0.3065870557744901" rpy="0 0 0"/>
+    <mass value="2.9385762719335418"/>
+    <inertia ixx="0.133646" iyy="0.133692" izz="0.00521" ixy="0.001039" iyz="-0.006152" ixz="0.011452"/>
+  </inertial>
+  <visual>
+    <origin xyz="-0.2675 0.32 -0.019" rpy="0 0 0"/>
     <geometry>
       <mesh filename="package://robotic_arm_description/meshes/camera_support.stl" scale="0.001 0.001 0.001"/>
     </geometry>
-    <material name="pa_12_nylon_pa_603cf_with_eos_p_3d_printers"/>
-  </visual>
-  <collision>
-    <origin xyz="-0.0 0.325 -0.02" rpy="0 0 0"/>
+    <material name="black_3d_printed"/>
+  </visual>
+  <collision>
+    <origin xyz="-0.2675 0.32 -0.019" rpy="0 0 0"/>
     <geometry>
       <mesh filename="package://robotic_arm_description/meshes/camera_support.stl" scale="0.001 0.001 0.001"/>
     </geometry>
   </collision>
+</link>
+<link name="camera_link">
+  <inertial>
+    <origin xyz="-2.682209454540896e-10 4.349266702619037e-07 -0.0009999921768903963" rpy="0 0 0"/>
+    <mass value="0.006279999999999998"/>
+    <inertia ixx="0.0" iyy="0.0" izz="0.0" ixy="0.0" iyz="0.0" ixz="-0.0"/>
+  </inertial>
+  <visual>
+    <origin xyz="-0.2245 0.249302 -0.53399" rpy="0 0 0"/>
+    <geometry>
+      <mesh filename="package://robotic_arm_description/meshes/camera_link.stl" scale="0.001 0.001 0.001"/>
+    </geometry>
+    <material name="steel_satin"/>
+  </visual>
+  <collision>
+    <origin xyz="-0.2245 0.249302 -0.53399" rpy="0 0 0"/>
+    <geometry>
+      <mesh filename="package://robotic_arm_description/meshes/camera_link.stl" scale="0.001 0.001 0.001"/>
+    </geometry>
+  </collision>
+</link>
+<link name="camera_link_frame">
 </link>
 <link name="base">
@@ -125,5 +147,5 @@
       <mesh filename="package://robotic_arm_description/meshes/base.stl" scale="0.001 0.001 0.001"/>
     </geometry>
-    <material name="pa_12_nylon_pa_603cf_with_eos_p_3d_printers"/>
+    <material name="black_3d_printed"/>
   </visual>
   <collision>
@@ -145,5 +167,5 @@
       <mesh filename="package://robotic_arm_description/meshes/waist.stl" scale="0.001 0.001 0.001"/>
     </geometry>
-    <material name="pa_12_nylon_pa_603cf_with_eos_p_3d_printers"/>
+    <material name="black_3d_printed"/>
   </visual>
   <collision>
@@ -165,5 +187,5 @@
       <mesh filename="package://robotic_arm_description/meshes/link_1.stl" scale="0.001 0.001 0.001"/>
     </geometry>
-    <material name="pa_12_nylon_pa_603cf_with_eos_p_3d_printers"/>
+    <material name="black_3d_printed"/>
   </visual>
   <collision>
@@ -185,5 +207,5 @@
       <mesh filename="package://robotic_arm_description/meshes/link_2.stl" scale="0.001 0.001 0.001"/>
     </geometry>
-    <material name="pa_12_nylon_pa_603cf_with_eos_p_3d_printers"/>
+    <material name="black_3d_printed"/>
   </visual>
   <collision>
@@ -205,5 +227,5 @@
       <mesh filename="package://robotic_arm_description/meshes/gripper_base.stl" scale="0.001 0.001 0.001"/>
     </geometry>
-    <material name="pa_12_nylon_pa_603cf_with_eos_p_3d_printers"/>
+    <material name="black_3d_printed"/>
   </visual>
   <collision>
@@ -225,5 +247,5 @@
       <mesh filename="package://robotic_arm_description/meshes/gripper_finger_1.stl" scale="0.001 0.001 0.001"/>
     </geometry>
-    <material name="pa_12_nylon_pa_603cf_with_eos_p_3d_printers"/>
+    <material name="black_3d_printed"/>
   </visual>
   <collision>
@@ -245,5 +267,5 @@
       <mesh filename="package://robotic_arm_description/meshes/gripper_finger_2.stl" scale="0.001 0.001 0.001"/>
     </geometry>
-    <material name="pa_12_nylon_pa_603cf_with_eos_p_3d_printers"/>
+    <material name="black_3d_printed"/>
   </visual>
   <collision>
@@ -280,7 +302,17 @@
 </joint>
 <joint name="rigid_5" type="fixed">
-  <origin xyz="0.0 -0.325 0.02" rpy="0 0 0"/>
+  <origin xyz="0.2375 -0.32 0.019" rpy="0 0 0"/>
   <parent link="base_link"/>
   <child link="camera_support"/>
+</joint>
+<joint name="camera_joint" type="fixed">
+  <origin xyz="-0.043 0.070698 0.51499" rpy="0 0 0"/>
+  <parent link="camera_support"/>
+  <child link="camera_link"/>
+</joint>
+<joint name="camera_link_frame_joint" type="fixed">
+  <origin xyz="0.01 0.0 0.0" rpy="0 0 0"/>
+  <parent link="camera_link"/>
+  <child link="camera_link_frame"/>
 </joint>
 <joint name="base_waist_joint" type="revolute">

File: robotic_arm_description/urdf/robotic_arm_gazebo.xacro (robot description, xacro)
@@ -7,6 +7,7 @@
 <xacro:property name="gripper_base_color" value = "Gazebo/FlatBlack" />
 <xacro:property name="gripper_gears" value="Gazebo/Blue"/>
-<xacro:property name="camera_color" value="Gazebo/WoodFloor" />
+<xacro:property name="camera_support_color" value="Gazebo/WoodFloor" />
 <xacro:property name="container_color" value="Gazebo/Red" />
+<xacro:property name="camera_color" value="Gazebo/Silver" />
   <gazebo reference="base_link">
     <material>${base_color}</material>
@@ -59,4 +60,10 @@
   </gazebo>
   <gazebo reference="camera_support">
+    <material>${camera_support_color}</material>
+    <mu1>0.2</mu1>
+    <mu2>0.2</mu2>
+    <self_collide>true</self_collide>
+  </gazebo>
+  <gazebo reference="camera_link">
     <material>${camera_color}</material>
     <mu1>0.2</mu1>
