Commit message: added arduino sketch for communication with ros,2, updated controllers

File: robotic_arm_description/urdf/robotic_arm.xacro (robot description, xacro)
@@ -1,4 +1,6 @@
 <?xml version="1.0" ?>
 <robot name="robotic_arm" xmlns:xacro="http://www.ros.org/wiki/xacro">
+<!-- Load Simulated or Real Hardware Interfaces -->
+<xacro:arg name="is_sim" default="true"/>
 <xacro:include filename="$(find robotic_arm_description)/urdf/materials.xacro" />
 <xacro:include filename="$(find robotic_arm_description)/urdf/robotic_arm.trans" />
@@ -6,5 +8,5 @@
 <xacro:include filename="$(find robotic_arm_description)/urdf/robotic_arm_controllers.xacro"/>
 <!-- Properties -->
-<xacro:property name="PI" value="1.570796"/>
+<xacro:property name="PI" value="1.570796"/>\
 <!-- Links -->
 <link name = "world"/>

File: robotic_arm_description/urdf/robotic_arm_controllers.xacro (robot description, xacro)
@@ -3,8 +3,17 @@
 <xacro:property name="gripper_angle" value="0.7854"/>
 <xacro:property name="PI" value="3.14159"/>
-<ros2_control type = "system" name = "RoboticArmSystem">
+<xacro:if value = "$(arg is_sim)">
     <hardware>
         <plugin>gazebo_ros2_control/GazeboSystem</plugin>
     </hardware>
+</xacro:if>
+<xacro:unless value = "$(arg is_sim)">
+    <hardware>
+        <plugin>robotic_arm_hw/RoboticArmHWInterface</plugin>
+        <!-- Change the port here -->
+        <param name ="port">/dev/ttyUSB0</param>
+    </hardware>
+</xacro:unless>
+<ros2_control type = "system" name = "RoboticArmSystem">
 <!-- Interfaces -->
     <joint name="base_waist_joint">

Commit message: hardware interface update

File: robotic_arm_description/urdf/robotic_arm.xacro (robot description, xacro)
@@ -1,9 +1,13 @@
-<?xml version="1.0" ?>
+<?xml version="1.0" encoding = "UTF-8"?>
 <robot name="robotic_arm" xmlns:xacro="http://www.ros.org/wiki/xacro">
 <!-- Load Simulated or Real Hardware Interfaces -->
+<xacro:arg name="sim_mode" default="true"/>
+<!-- Include materials properties to be used with rviz -->
 <xacro:include filename="$(find robotic_arm_description)/urdf/materials.xacro" />
 <xacro:include filename="$(find robotic_arm_description)/urdf/robotic_arm.trans" />
+<!-- Include material properties to be used in gazebo -->
 <xacro:include filename="$(find robotic_arm_description)/urdf/robotic_arm_gazebo.xacro"/>
-<xacro:include filename="$(find robotic_arm_description)/urdf/robotic_arm_controllers.xacro"/>
+<!-- Include ros2_control plugin-->
+<xacro:include filename="$(find robotic_arm_description)/urdf/robotic_arm_ros2_control.xacro"/>
 <!-- Properties -->
 <xacro:property name="PI" value="1.570796"/>
@@ -30,5 +34,5 @@
   </collision>
 </link>
-<link name="container_1">
+<link name="container_cubes">
   <inertial>
     <origin xyz="0.0021344768560282723 -1.5647124724599282e-05 0.026103286200414536" rpy="0 0 0"/>
@@ -39,5 +43,5 @@
     <origin xyz="0.2025 0.225 -0.035" rpy="0 0 0"/>
     <geometry>
-      <mesh filename="package://robotic_arm_description/meshes/container_1.stl" scale="0.001 0.001 0.001"/>
+      <mesh filename="package://robotic_arm_description/meshes/container_cubes.stl" scale="0.001 0.001 0.001"/>
     </geometry>
     <material name="led_red"/>
@@ -46,9 +50,9 @@
     <origin xyz="0.2025 0.225 -0.035" rpy="0 0 0"/>
     <geometry>
-      <mesh filename="package://robotic_arm_description/meshes/container_1.stl" scale="0.001 0.001 0.001"/>
-    </geometry>
-  </collision>
-</link>
-<link name="container_2">
+      <mesh filename="package://robotic_arm_description/meshes/container_cubes.stl" scale="0.001 0.001 0.001"/>
+    </geometry>
+  </collision>
+</link>
+<link name="container_cylinders">
   <inertial>
     <origin xyz="-1.565155782010108e-05 -0.0021344802460424653 0.026103286200414424" rpy="0 0 0"/>
@@ -59,5 +63,5 @@
     <origin xyz="0.2425 0.02 -0.035" rpy="0 0 0"/>
     <geometry>
-      <mesh filename="package://robotic_arm_description/meshes/container_2.stl" scale="0.001 0.001 0.001"/>
+      <mesh filename="package://robotic_arm_description/meshes/container_cylinders.stl" scale="0.001 0.001 0.001"/>
     </geometry>
     <material name="led_red"/>
@@ -66,9 +70,9 @@
     <origin xyz="0.2425 0.02 -0.035" rpy="0 0 0"/>
     <geometry>
-      <mesh filename="package://robotic_arm_description/meshes/container_2.stl" scale="0.001 0.001 0.001"/>
-    </geometry>
-  </collision>
-</link>
-<link name="container_3">
+      <mesh filename="package://robotic_arm_description/meshes/container_cylinders.stl" scale="0.001 0.001 0.001"/>
+    </geometry>
+  </collision>
+</link>
+<link name="container_hexagons">
   <inertial>
     <origin xyz="-1.565155782010108e-05 -0.0021344802460424445 0.0261032862004145" rpy="0 0 0"/>
@@ -79,5 +83,5 @@
     <origin xyz="0.1375 0.02 -0.035" rpy="0 0 0"/>
     <geometry>
-      <mesh filename="package://robotic_arm_description/meshes/container_3.stl" scale="0.001 0.001 0.001"/>
+      <mesh filename="package://robotic_arm_description/meshes/container_hexagons.stl" scale="0.001 0.001 0.001"/>
     </geometry>
     <material name="led_red"/>
@@ -86,5 +90,5 @@
     <origin xyz="0.1375 0.02 -0.035" rpy="0 0 0"/>
     <geometry>
-      <mesh filename="package://robotic_arm_description/meshes/container_3.stl" scale="0.001 0.001 0.001"/>
+      <mesh filename="package://robotic_arm_description/meshes/container_hexagons.stl" scale="0.001 0.001 0.001"/>
     </geometry>
   </collision>
@@ -250,6 +254,6 @@
   </collision>
 </link>
+<!-- Joints -->
 <joint name = "virtual_joint" type= "fixed">
-  <origin xyz="0.0 0.0 0.0" rpy="0.0 0.0 0.0"/>
   <parent link="world"/>
   <child link="base_link"/>
@@ -263,15 +267,15 @@
   <origin xyz="-0.2025 -0.225 0.035" rpy="0 0 0"/>
   <parent link="base_link"/>
-  <child link="container_1"/>
+  <child link="container_cubes"/>
 </joint>
 <joint name="rigid_3" type="fixed">
   <origin xyz="-0.2425 -0.02 0.035" rpy="0 0 0"/>
   <parent link="base_link"/>
-  <child link="container_2"/>
+  <child link="container_cylinders"/>
 </joint>
 <joint name="rigid_4" type="fixed">
   <origin xyz="-0.1375 -0.02 0.035" rpy="0 0 0"/>
   <parent link="base_link"/>
-  <child link="container_3"/>
+  <child link="container_hexagons"/>
 </joint>
 <joint name="rigid_5" type="fixed">
@@ -301,5 +305,5 @@
   <limit upper="1.570796" lower="-1.570796" effort="100" velocity="100"/>
 </joint>
-<joint name="link2_gipper_base_joint" type="revolute">
+<joint name="link2_gripper_base_joint" type="revolute">
   <origin xyz="0.00385 -0.11735 0.0003" rpy="0 0 0"/>
   <parent link="link_2"/>
@@ -321,6 +325,6 @@
   <axis xyz="-0.0 0.0 1.0"/>
   <dynamics damping="10.0" friction="2.0"/>
-  <mimic joint = "right_gripper_joint" multiplier = "-1.0"/>
   <limit upper="0.0" lower="-1.047198" effort="100" velocity="100"/>
+  <mimic joint = "right_gripper_joint" multiplier = "-1"/>
 </joint>
 </robot>

File: robotic_arm_description/urdf/robotic_arm_gazebo.xacro (robot description, xacro)
@@ -1,12 +1,11 @@
 <?xml version="1.0" encoding = "UTF-8"?>
 <robot name="robotic_arm" xmlns:xacro="http://www.ros.org/wiki/xacro" >
-<xacro:property name="base_color" value = "Gazebo/Oak"/>
-<xacro:property name="waist_color" value = "Gazebo/FlatBlack" />
+<xacro:property name="base_color" value =  "Gazebo/Wood"/>
+<xacro:property name="waist_color" value = "Gazebo/FlatBlack"/>
 <xacro:property name="link_1_color" value = "Gazebo/FlatBlack"/>
 <xacro:property name="link_2_color" value = "Gazebo/FlatBlack" />
 <xacro:property name="gripper_base_color" value = "Gazebo/FlatBlack" />
-<xacro:property name="gripper_gears" value="GazeboGrey"/>
-<xacro:property name="gripper_color" value="Gazebo/DarkGrey"/>
-<xacro:property name="camera_color" value="Gazebo/Oak" />
+<xacro:property name="gripper_gears" value="Gazebo/Blue"/>
+<xacro:property name="camera_color" value="Gazebo/WoodFloor" />
 <xacro:property name="container_color" value="Gazebo/Red" />
   <gazebo reference="base_link">
@@ -65,5 +64,5 @@
     <self_collide>true</self_collide>
   </gazebo>
-  <gazebo reference="container_1">
+  <gazebo reference="container_cubes">
     <material>${container_color}</material>
     <mu1>0.2</mu1>
@@ -71,5 +70,5 @@
     <self_collide>true</self_collide>
   </gazebo>
-  <gazebo reference="container_2">
+  <gazebo reference="container_cylinders">
     <material>${container_color}</material>
     <mu1>0.2</mu1>
@@ -77,5 +76,5 @@
     <self_collide>true</self_collide>
   </gazebo>
-  <gazebo reference="container_3">
+  <gazebo reference="container_hexagons">
     <material>${container_color}</material>
     <mu1>0.2</mu1>

File: robotic_arm_description/urdf/robotic_arm_urdf.urdf (robot description, URDF)
Before this commit: robot robotic_arm, 9 links, 8 joints
Links:
- added link camera_support, mass 1.9073849170892592; collision mesh filename=package://robotic_arm_description/meshes/camera_support.stl scale=0.001 0.001 0.001; visual mesh filename=package://robotic_arm_description/meshes/camera_support.stl scale=0.001 0.001 0.001
- added link container_cubes, mass 0.8859344258495231; collision mesh filename=package://robotic_arm_description/meshes/container_cubes.stl scale=0.001 0.001 0.001; visual mesh filename=package://robotic_arm_description/meshes/container_cubes.stl scale=0.001 0.001 0.001
- added link container_cylinders, mass 0.8859344258495231; collision mesh filename=package://robotic_arm_description/meshes/container_cylinder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 scale=0.001 0.001 0.001; visual mesh filename=package://robotic_arm_description/meshes/container_cylinder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 scale=0.001 0.001 0.001
- added link container_hexagons, mass 0.8859344258495231; collision mesh filename=package://robotic_arm_description/meshes/container_hexagons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 scale=0.001 0.001 0.001; visual mesh filename=package://robotic_arm_description/meshes/container_hexagons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 scale=0.001 0.001 0.001
- link base_link: mass 2.5408670074548567 -> 2.562361438794821
Joints:
- added joint rigid_2: type fixed, parent base_link, child container_cubes, origin xyz=-0.2025 -0.225 0.035 rpy=0 0 0
- added joint rigid_3: type fixed, parent base_link, child container_cylinders, origin xyz=-0.2425 -0.02 0.035 rpy=0 0 0
- added joint rigid_4: type fixed, parent base_link, child container_hexagons, origin xyz=-0.1375 -0.02 0.035 rpy=0 0 0
- added joint rigid_5: type fixed, parent base_link, child camera_support, origin xyz=0.0 -0.325 0.02 rpy=0 0 0
- joint base_waist_joint: axis 0.0 0.0 1.0 -> -0.0 -0.0 1.0; origin xyz=-0.0 -0.07 0.086 rpy=0 0 0 -> xyz=-0.0 -0.08 0.086 rpy=0 0 0
- joint left_gripper_joint: axis 0.0 0.0 1.0 -> -0.0 0.0 1.0; child gripper_finger_1 -> gripper_finger_2; limit lower=0.0 upper=-0.785398 effort=100 velocity=100 -> lower=-1.047198 upper=0.0 effort=100 velocity=100; mimic joint=right_gripper_joint multiplier=1.0 -> joint=right_gripper_joint multiplier=-1; origin xyz=0.0259 -0.038 0.01535 rpy=0 0 0 -> xyz=-0.001 -0.038 0.014 rpy=0 0 0
- joint link1_link2_joint: axis -1.0 0.0 0.0 -> 1.0 -0.0 -0.0; limit lower=0.0 upper=3.141593 effort=100 velocity=100 -> lower=-1.570796 upper=1.570796 effort=100 velocity=100
- joint link2_gripper_base_joint: axis 1.0 0.0 0.0 -> 1.0 -0.0 0.0
- joint right_gripper_joint: axis 0.0 0.0 -1.0 -> -0.0 0.0 1.0; child gripper_finger_2 -> gripper_finger_1; limit lower=0.0 upper=0.785398 effort=100 velocity=100 -> lower=0.0 upper=1.047198 effort=100 velocity=100; origin xyz=-0.001 -0.038 0.014 rpy=0 0 0 -> xyz=0.0259 -0.038 0.014 rpy=0 0 0
- joint rigid_1: origin xyz=0.0 0.07 0.015 rpy=0 0 0 -> xyz=0.0 0.07 0.035 rpy=0 0 0
- joint virtual_joint: origin xyz=0.0 0.0 0.0 rpy=0.0 0.0 0.0 -> (none)
- joint waist_link1_joint: axis 1.0 0.0 0.0 -> 1.0 0.0 -0.0

Commit message: working code

File: robotic_arm_description/urdf/robotic_arm.xacro (robot description, xacro)
@@ -10,6 +10,8 @@
 <!-- Include ros2_control plugin-->
 <xacro:include filename="$(find robotic_arm_description)/urdf/robotic_arm_ros2_control.xacro"/>
+<!-- Include camera plugins -->
+<xacro:include filename="$(find robotic_arm_description)/urdf/robotic_arm_camera.xacro"/>
 <!-- Properties -->
-<xacro:property name="PI" value="1.570796"/>
+<xacro:property name="PI" value="3.147"/>
 <!-- Links -->
 <link name = "world"/>
@@ -312,5 +314,5 @@
 </joint>
 <joint name="camera_link_frame_joint" type="fixed">
-  <origin xyz="0.01 0.0 0.0" rpy="0 0 0"/>
+  <origin xyz="0.0 0.0 0.0" rpy="3.14 1.57 0"/>
   <parent link="camera_link"/>
   <child link="camera_link_frame"/>

File: robotic_arm_description/urdf/robotic_arm_camera.xacro (robot description, xacro)
@@ -1,2 +1,3 @@
+<?xml version="1.0" encoding = "UTF-8"?>
 <robot xmlns:xacro="http://www.ros.org/wiki/xacro" name="robotic_arm">
     <!-- Camera -->
@@ -4,8 +5,9 @@
     <sensor type="camera" name="rgb_cam">
       <always_on>1</always_on>
+      <pose>0 0 0 0 0 0</pose>
+      <visualize>true</visualize>
       <update_rate>10.0</update_rate>
       <camera name="rgb_cam">
-          <pose>0 0 0 0 0 0</pose>
-          <horizontal_fov>1.3962634</horizontal_fov>
+          <horizontal_fov>1.396264</horizontal_fov>
           <image>
            <width>640</width>
@@ -14,6 +16,6 @@
           </image>
           <clip>
-              <near>0.005</near>
-              <far>20.0</far>
+              <near>0.05</near>
+              <far>8.0</far>
           </clip>
       </camera>

Commit message: integration of the webcam with ros2

File: robotic_arm_description/urdf/robotic_arm.xacro (robot description, xacro)
@@ -314,5 +314,5 @@
 </joint>
 <joint name="camera_link_frame_joint" type="fixed">
-  <origin xyz="0.0 0.0 0.0" rpy="3.14 1.57 0"/>
+  <origin xyz="0.0 0.0 0.0" rpy="${PI} ${PI/2} 0"/>
   <parent link="camera_link"/>
   <child link="camera_link_frame"/>

File: robotic_arm_description/urdf/robotic_arm_camera.xacro (robot description, xacro)
@@ -9,5 +9,5 @@
       <update_rate>10.0</update_rate>
       <camera name="rgb_cam">
-          <horizontal_fov>1.396264</horizontal_fov>
+          <horizontal_fov>1.234</horizontal_fov>
           <image>
            <width>640</width>
@@ -17,5 +17,5 @@
           <clip>
               <near>0.05</near>
-              <far>8.0</far>
+              <far>1.0</far>
           </clip>
       </camera>

File: robotic_arm_description/urdf/robotic_arm_ros2_control.xacro (robot description, xacro)
@@ -62,5 +62,5 @@
         <plugin>robotic_arm_controllers/RoboticArmHWInterface</plugin>
         <param name="port_">/dev/ttyUSB0</param>
-        <param name="baud_rate">115200</param>
+        <param name="baud_rate">9600</param>
     </hardware>
     <!-- Interfaces -->

File: robotic_arm_description/urdf/robotic_arm_urdf.urdf (robot description, URDF)
Before this commit: robot robotic_arm, 12 links, 11 joints
Joints:
- joint end_effector_link: origin xyz= 0 -0.08 0  rpy=0 0 0 -> xyz= 0.01 -0.08 0.01  rpy=0 0 0

Commit message: push for kevin

File: robotic_arm_description/urdf/robotic_arm.xacro (robot description, xacro)
@@ -12,8 +12,10 @@
 <!-- Include camera plugins -->
 <xacro:include filename="$(find robotic_arm_description)/urdf/robotic_arm_camera.xacro"/>
+<!-- Links -->
+<link name = "world"/>
+<!--include aruco marke-->
+<xacro:include filename="$(find robotic_arm_description)/urdf/aruco_marker.xacro"/>
 <!-- Properties -->
 <xacro:property name="PI" value="3.147"/>
-<!-- Links -->
-<link name = "world"/>
 <link name="base_link">
   <inertial>

File: robotic_arm_description/urdf/robotic_arm_urdf.urdf (robot description, URDF)
Before this commit: robot robotic_arm, 12 links, 11 joints
Links:
- link gripper_base: geometry collision box size=0.01 0.1 0.01; visual box size=0.01 0.1 0.01
Joints:
- joint end_effector_link: origin xyz= 0.01 -0.08 0.01  rpy=0 0 0 -> xyz= 0.01 -0.1 0.01  rpy=0 0 0
